File: adp5350_example/adp5350_devboard/_saved_adp5350_devboard.sch (KiCad schematic (older format))
At the start: 46 parts, among them J2 Conn_01x11, U1 adp5350

Commit message: Mapped schematic parts to footprints for PCB. Size of L/R/C footprints -> 1206
Simplified some circuitry for the sake of sizing and uneeded parts.
Changed test points out with individual parts.
2 errors in electrical rules/connectivity testing ignored (not important)
Parts:
- gave numbers to parts that had none: 1
Changed lines of the file:
@@
 Connection ~ 7050 2500
 $Comp
-L Conn_01x03 J?
+L Conn_01x03 J1
 U 1 1 5A04CC65
 P 1700 4100
-F 0 "J?" H 1700 4300 50  0000 C CNN
+F 0 "J1" H 1700 4300 50  0000 C CNN
 F 1 "Conn_01x03" H 1700 3900 50  0000 C CNN
 F 2 "" H 1700 4100 50  0001 C CNN
@@
 	1950 4200 1950 4250
 $Comp
-L GND #PWR?
+L GND #PWR025
 U 1 1 5A04DD19
 P 1950 4250
-F 0 "#PWR?" H 1950 4000 50  0001 C CNN
+F 0 "#PWR025" H 1950 4000 50  0001 C CNN
 F 1 "GND" H 1950 4100 50  0000 C CNN
 F 2 "" H 1950 4250 50  0001 C CNN
